Commit message: Add content to ros2_ws

File: ros2_ws/src/my_robot/urdf/my_robot.urdf (robot description, URDF)
Before this commit: robot my_robot, 1 links, 0 joints
Links:
- added link right_leg; visual box size=0.6 0.1 0.2
Joints:
- added joint base_to_right_leg: type continuous, parent base_link, child right_leg, origin xyz=0 -0.22 0.25, axis 0 1 0
