Commit message: Add content to ros2_ws

File: ros2_ws/src/my_robot/urdf/my_conveyor_belt.xacro (robot description, xacro)
@@ -1,26 +1,27 @@
 <?xml version="1.0"?>
-<robot xmlns:xacro="http://www.ros.org/wiki/xacro" name="my_conveyor_belt">
-    <!-- Material definitions -->
-    <material name="grey">
+<robot xmlns:xacro="http://www.ros.org/wiki/xacro" name="my_conveyor_belt_robot">
+    <xacro:property name="base_length" value="2.4"/>
+    <xacro:property name="base_width" value="0.4"/>
+    <xacro:property name="base_height" value="0.2"/>
+    <xacro:property name="axle_length" value="0.15"/>
+    <xacro:property name="axle_width" value="0.10"/>
+    <xacro:property name="axle_height" value="0.06"/>
+    <xacro:property name="arm_length" value="0.55"/>
+    <xacro:property name="arm_width" value="0.10"/>
+    <xacro:property name="arm_height" value="0.06"/>
+    <xacro:property name="axle_spacing" value="0.65"/>
+    <xacro:property name="pi_" value="3.14159265359"/>
+    <!-- Materials -->
+    <material name="gray">
         <color rgba="0.5 0.5 0.5 1.0"/>
     </material>
-    <material name="white">
-        <color rgba="1.0 1.0 1.0 1.0"/>
+    <material name="yellow">
+        <color rgba="1.0 1.0 0.0 1.0"/>
     </material>
     <material name="black">
         <color rgba="0.0 0.0 0.0 1.0"/>
     </material>
-    <!-- Link properties -->
-    <xacro:property name="base_length" value="2.0"/>
-    <xacro:property name="base_width" value="0.5"/>
-    <xacro:property name="base_height" value="0.2"/>
-    <xacro:property name="bar_length" value="0.6"/>
-    <xacro:property name="bar_width" value="0.2"/>
-    <xacro:property name="bar_height" value="0.1"/>
-    <xacro:property name="sphere_radius" value="0.05"/>
-    <xacro:property name="sphere_offset" value="0.4"/>
-    <xacro:property name="pi_" value="3.14159265359"/>
-    <!-- Predefine links -->
-    <xacro:macro name="bar_link" params="name length width height material">
+    <!-- Macros for Links -->
+    <xacro:macro name="box_link" params="name length width height material">
         <link name="${name}">
             <visual>
@@ -28,5 +29,5 @@
                     <box size="${length} ${width} ${height}"/>
                 </geometry>
-                <origin rpy="0 0 0" xyz="0 0 0"/>
+                <origin rpy="0 0 0" xyz="${-length/2} 0 0"/>
                 <material name="${material}"/>
             </visual>
@@ -35,25 +36,10 @@
                     <box size="${length} ${width} ${height}"/>
                 </geometry>
-                <origin rpy="0 0 0" xyz="0 0 0"/>
+                <origin rpy="0 0 0" xyz="${-length/4} 0 0"/>
             </collision>
+            <inertial> <mass value="0.1"/> <inertia ixx="0.001" ixy="0" ixz="0" iyy="0.001" iyz="0" izz="0.001"/> </inertial>
         </link>
     </xacro:macro>
-    <xacro:macro name="sphere_link" params="name radius material">
-        <link name="${name}">
-            <visual>
-                <geometry>
-                    <sphere radius="${radius}"/>
-                </geometry>
-                <origin rpy="0 0 0" xyz="0 0 0"/>
-                <material name="${material}"/>
-            </visual>
-            <collision>
-                <geometry>
-                    <sphere radius="${radius}"/>
-                </geometry>
-                <origin rpy="0 0 0" xyz="0 0 0"/>
-            </collision>
-        </link>
-    </xacro:macro>
+    <!-- Macros for Joints -->
     <xacro:macro name="fixed_joint" params="name parent child x y z">
         <joint name="${name}" type="fixed">
@@ -63,27 +49,108 @@
         </joint>
     </xacro:macro>
-    <xacro:macro name="revolute_joint" params="name parent child x y z lower_limit upper_limit">
-        <joint name="${name}" type="revolute">
+    <xacro:macro name="revolute_joint" params="name parent child x y z rpy lower_limit upper_limit axis">
+         <joint name="${name}" type="revolute">
             <parent link="${parent}"/>
             <child link="${child}"/>
-            <origin xyz="${x} ${y} ${z}" rpy="0 0 0"/>
-            <axis xyz="0 0 1"/>
-            <limit lower="${lower_limit}" upper="${upper_limit}" effort="100" velocity="10"/>
+            <origin xyz="${x} ${y} ${z}" rpy="${rpy}"/>
+            <axis xyz="${axis}"/>
+            <limit lower="${lower_limit}" upper="${upper_limit}" effort="100" velocity="2"/>
         </joint>
     </xacro:macro>
-    <!-- Call macros -->
-    <xacro:bar_link name="base_link" length="${base_length}" width="${base_width}" height="${base_height}" material="grey"/>
-    <!-- Joints -->
-    <xacro:macro name="axle_and_bar" params="index">
-        <xacro:property name="x_pos" value="${-base_length/2 + sphere_offset * (index + 0.5)}"/>
-        <xacro:sphere_link name="axle_${index}" radius="${sphere_radius}" material="black"/>
-        <xacro:fixed_joint name="base_to_axle_${index}" parent="base_link" child="axle_${index}" x="${x_pos}" y="0" z="${-base_height/2 - sphere_radius}"/>
-        <xacro:bar_link name="bar_${index}" length="${bar_length}" width="${bar_width}" height="${bar_height}" material="white"/>
-        <xacro:revolute_joint name="axle_${index}_to_bar_${index}" parent="axle_${index}" child="bar_${index}" x="0" y="0" z="${-sphere_radius - bar_height/2}" lower_limit="${-pi_/4}" upper_limit="${pi_/4}"/>
+    <!-- World Link and Joint to ground the robot -->
+    <link name="world"/>
+    <joint name="world_joint" type="fixed">
+        <parent link="world"/>
+        <child link="base_link"/>
+        <origin xyz="0 0 ${arm_height + axle_height + base_height/2}" rpy="0 0 0"/>
+    </joint>
+    <!-- Base Link -->
+    <xacro:box_link name="base_link" length="${base_length}" width="${base_width}" height="${base_height}" material="gray"/>
+    <!-- Macro for Axle and Bar unit -->
+    <xacro:macro name="axle_and_arm" params="index">
+        <xacro:property name="x_pos" value="${-base_length + axle_spacing * (index + 0.6)}"/>
+        <xacro:box_link name="axle_${index}" length="${axle_length}" width="${axle_width}" height="${axle_height}" material="yellow"/>
+        <xacro:fixed_joint name="base_to_axle_${index}" parent="base_link" child="axle_${index}"
+                           x="${x_pos}" y="${-base_width/2 - axle_width/2}" z="${-base_height/2 + axle_height/2}"/>
+        <!-- Arm (Box) Link -->
+        <xacro:box_link name="arm_${index}" length="${arm_length}" width="${arm_width}" height="${arm_height}" material="black"/>
+        <!-- Joint: Axle Link to Bar Link (Revolute) -->
+        <xacro:revolute_joint name="axle_${index}_to_arm_${index}"
+                              parent="axle_${index}"
+                              child="arm_${index}"
+                              x="${-axle_length/3}"
+                              y="0"
+                              z="${-axle_height}"
+                              rpy="0 0 0"
+                              lower_limit="0"
+                              upper_limit="${pi_/4}"
+                              axis="0 0 1"
+                              />
     </xacro:macro>
-    <!-- Call joints -->
-    <xacro:axle_and_bar index="0"/>
-    <xacro:axle_and_bar index="1"/>
-    <xacro:axle_and_bar index="2"/>
-    <xacro:axle_and_bar index="3"/>
+    <!-- Create 4 units -->
+    <xacro:axle_and_arm index="0"/>
+    <xacro:axle_and_arm index="1"/>
+    <xacro:axle_and_arm index="2"/>
+    <xacro:axle_and_arm index="3"/>
+<!-- Plugin Gazebo Classic -->
+  <gazebo>
+    <plugin name="gazebo_ros2_control" filename="libgazebo_ros2_control.so">
+      <robot_namespace>my_conveyor_belt_robot</robot_namespace>
+      <parameters>/home/admin1/ros2_ws/install/my_conveyor_gazebo/share/my_conveyor_gazebo/config/controllers.yaml</parameters>
+    </plugin>
+  </gazebo>
+  <!-- ROS 2 Control hardware interface -->
+  <ros2_control name="GazeboSystem" type="system">
+    <hardware>
+      <plugin>gazebo_ros2_control/GazeboSystem</plugin>
+    </hardware>
+    <joint name="axle_0_to_arm_0">
+      <command_interface name="position"/>
+      <state_interface name="position"/>
+      <state_interface name="velocity"/>
+    </joint>
+    <joint name="axle_1_to_arm_1">
+      <command_interface name="position"/>
+      <state_interface name="position"/>
+      <state_interface name="velocity"/>
+    </joint>
+    <joint name="axle_2_to_arm_2">
+      <command_interface name="position"/>
+      <state_interface name="position"/>
+      <state_interface name="velocity"/>
+    </joint>
+    <joint name="axle_3_to_arm_3">
+      <command_interface name="position"/>
+      <state_interface name="position"/>
+      <state_interface name="velocity"/>
+    </joint>
+  </ros2_control>
+  <!-- Gazebo Material -->
+  <gazebo reference="base_link">
+    <material>Gazebo/Grey</material>
+  </gazebo>
+  <gazebo reference="axle_0">
+    <material>Gazebo/Yellow</material>
+  </gazebo>
+  <gazebo reference="axle_1">
+    <material>Gazebo/Yellow</material>
+  </gazebo>
+  <gazebo reference="axle_2">
+    <material>Gazebo/Yellow</material>
+  </gazebo>
+  <gazebo reference="axle_3">
+    <material>Gazebo/Yellow</material>
+  </gazebo>
+  <gazebo reference="arm_0">
+    <material>Gazebo/Black</material>
+  </gazebo>
+  <gazebo reference="arm_1">
+    <material>Gazebo/Black</material>
+  </gazebo>
+  <gazebo reference="arm_2">
+    <material>Gazebo/Black</material>
+  </gazebo>
+  <gazebo reference="arm_3">
+    <material>Gazebo/Black</material>
+  </gazebo>
 </robot>
