Commit message: add trash bin + finish the whole system

File: wc_ws/src/camera/yolobot_description/robot/yolobot.urdf (robot description, URDF)
Before this commit: robot yolobot, 4 links, 3 joints
Joints:
- joint rgb_cam_camera_link_joint: origin xyz=0.0 -2.4 1.55 rpy=0 0 0 -> xyz=0.0 -3.0 1.55 rpy=0 0 0
